File: hardware/antennaanalyzernx.sch (KiCad schematic (older format))
At the start: 140 parts, among them J1 Power Connection, J2 SPI Header, J3 Serial Header, J4 GPIO, J5 Conn_Coaxial, J6 TFT Connection, J7 Touch Connection, J8 SD Connection, SW1 Reset, U1 SA612, U10 TLV1117-33, U11 TLV1117-50, U12 ATmega1284P-AU, U2 LM358, U3 Si5351A, U4 SA612, U5 LM358, U6 74HC86, U7 74HC74, U8 LM358, U9 LM324, Y1 27MHz, Y2 16MHz

Commit message: stm32 version
Parts:
- removed C19, C2, C20, C27, C43: 100n, Capacitors_SMD:C_0805_HandSoldering, symbol Device:C
- removed C35, C36: 22p, Capacitors_SMD:C_0805_HandSoldering, symbol Device:C
- removed D1, D2: 1n4148, Diodes_SMD:D_SOD-323, symbol Device:D
- removed J2: SPI Header, Connectors_Molex:Molex_KK-6410-04_04x2.54mm_Straight, symbol Connector:Conn_01x04_Female
- removed J3: Serial Header, Connectors_Molex:Molex_KK-6410-06_06x2.54mm_Straight, symbol Connector:Conn_01x06_Female
- removed J4: GPIO, Connectors_Molex:Molex_KK-6410-04_04x2.54mm_Straight, symbol Connector:Conn_01x04_Female
- removed J6: TFT Connection, Connectors_Molex:Molex_KK-6410-09_09x2.54mm_Straight, symbol Connector:Conn_01x09_Female
- removed J7: Touch Connection, Connectors_Molex:Molex_KK-6410-05_05x2.54mm_Straight, symbol Connector:Conn_01x05_Female
- removed L4: 1u, Inductors_SMD:L_1210_HandSoldering, symbol Device:L
- removed R1, R10, R34, R39, R40, R6: 10k, Resistors_SMD:R_0805_HandSoldering, symbol Device:R
- removed R13: 1k, Resistors_SMD:R_0805_HandSoldering, symbol Device:R
- removed RV1, RV2, RV3: 100k, Potentiometers:Potentiometer_Trimmer_Bourns_3266W, symbol Device:R_POT
- removed TP1: VV Test Point, Measurement_Points:Measurement_Point_Round-SMD-Pad_Small, symbol Connector:TestPoint
- removed TP2, TP3: TestPoint, Measurement_Points:Measurement_Point_Round-SMD-Pad_Small, symbol Connector:TestPoint
- removed U12: ATmega1284P-AU, Housings_QFP:TQFP-44_10x10mm_Pitch0.8mm, symbol MCU_Microchip_ATmega:ATmega1284P-AU
- removed U2, U5, U8: LM358, Housings_SOIC:SOIC-8_3.9x4.9mm_Pitch1.27mm, symbol Amplifier_Operational:LM358
- removed U6: 74HC86, Housings_SOIC:SOIC-14_3.9x8.7mm_Pitch1.27mm, symbol 74xx:74HC86
- removed U7: 74HC74, Housings_SOIC:SOIC-14_3.9x8.7mm_Pitch1.27mm, symbol 74xx:74HC74
- removed U9: LM324, Housings_SOIC:SOIC-14_3.9x8.7mm_Pitch1.27mm, symbol Amplifier_Operational:LM324
- added C10: 2.2u, Capacitors_SMD:C_0805_HandSoldering, symbol Device:C
- added C13, C15, C16, C17, C26, C29: 100n, Capacitors_SMD:C_0805_HandSoldering, symbol Device:C
- added C23, C24: 4.7u, Capacitors_SMD:C_0805_HandSoldering, symbol Device:C
- added C32: 20p, Capacitors_SMD:C_0805_HandSoldering, symbol Device:C
- added J1: USB_B_Micro, AntennaAnalyzer:USB Micro, symbol Connector:USB_B_Micro
- added J3: Conn_01x08_Male, Pin_Headers:Pin_Header_Straight_1x08_Pitch2.54mm, symbol Connector:Conn_01x08_Male
- added J4: TFT Header, Pin_Headers:Pin_Header_Straight_1x14_Pitch2.54mm, symbol Connector:Conn_01x14_Female
- added J7: Serial Header, Pin_Headers:Pin_Header_Straight_1x03_Pitch2.54mm, symbol Connector:Conn_01x03_Male
- added R17, R18, R19, R8, R9: 10k, Resistors_SMD:R_0805_HandSoldering, symbol Device:R
- added R21: 33, Resistors_SMD:R_0805_HandSoldering, symbol Device:R
- added SW2: SW_Push, AntennaAnalyzer:Switch, symbol Switch:SW_Push
- added U4: STM32F407VGTx, Housings_QFP:LQFP-100_14x14mm_Pitch0.5mm, symbol MCU_ST_STM32F4:STM32F407VGTx
- added U5: MCP602, Housings_SOIC:SOIC-8_3.9x4.9mm_Pitch1.27mm, symbol Amplifier_Operational:MCP602
- added U6: MCP604, Housings_SOIC:SOIC-14_3.9x8.7mm_Pitch1.27mm, symbol Amplifier_Operational:MCP604
- C14: value 10u -> 100n
- C21, C25: value 100n -> 1u
- C22: value 1u -> 100n
- C31: value 100n -> 20p
- C8: value 100n -> 10n
- C9: value 10u -> 2.2u
- J5: renamed from J1; footprint Connectors_Molex:Molex_KK-6410-02_02x2.54mm_Straight -> Pin_Headers:Pin_Header_Straight_1x02_Pitch2.54mm
- J6: renamed from J8; value SD Connection -> SD Header; footprint Connectors_Molex:Molex_KK-6410-04_04x2.54mm_Straight -> Pin_Headers:Pin_Header_Straight_1x04_Pitch2.54mm
- R3: value 10k -> 0
- SW1: value Reset -> SW_Push; footprint SMA:Switch -> AntennaAnalyzer:Switch
- U1: symbol sa612:SA612 -> antennaanalyzernx-rescue:SA612-sa612
- U2: renamed from U3; symbol SiLabs:Si5351A -> antennaanalyzernx-rescue:Si5351A-SiLabs
- U3: renamed from U4; symbol sa612:SA612 -> antennaanalyzernx-rescue:SA612-sa612
- Y2: value 16MHz -> Crystal
- renumbered C5 to C1, C13 to C11, C16 to C18, C17 to C19, C3 to C2, C18 to C20, C23 to C27, C24 to C28, C4 to C3, C26 to C30, C28 to C33, C29 to C34, C30 to C35, C32 to C36, C33 to C37, C34 to C38, C37 to C39, C1 to C4, C38 to C40, C39 to C41, C40 to C42, C41 to C43, C42 to C44, C44 to C45, C45 to C46, C46 to C47, C47 to C48, C48 to C49, C6 to C5, C49 to C50, C50 to C51, C51 to C52, C7 to C6, C10 to C7, D7 to D1, D8 to D2, D9 to D3, D3 to D4, D4 to D5, D5 to D6, D6 to D7, J5 to J2, R2 to R1, R11 to R10, R12 to R11, R43 to R12, R44 to R13, R45 to R14, R14 to R15, R15 to R16, R4 to R2, R41 to R20, R16 to R22, R17 to R23, R18 to R24, R19 to R25, R20 to R26, R21 to R27, R22 to R28, R23 to R29, R24 to R30, R25 to R31, R26 to R32, R42 to R33, R27 to R34, R28 to R35, R29 to R36, R30 to R37, R31 to R38, R32 to R39, R5 to R4, R33 to R40, R35 to R41, R36 to R42, R37 to R43, R38 to R44, R7 to R5, R8 to R6, R9 to R7, TP4 to TP1, TP5 to TP2, U10 to U7, U11 to U8
Connections:
- net 3.3V: now also C12.1, C14.1, C21.1, C22.1, C25.1, C36.2, R20.1, R27.1, R33.1, C13.1, C15.1, C16.1, C17.1, C23.1, C24.1, C26.1, J4.14 (Pin_14), R17.1, R21.2, U4.100 (VDD), U4.11 (VDD), U4.19 (VDD), U4.21 (VREF+), U4.22 (VDDA), U4.28 (VDD), U4.50 (VDD), U4.6 (VBAT), U4.75 (VDD), U5.8 (V+), U6.4 (V+)
- net 5V: no longer C21.2, C25.1, C36.2, C8.2, R20.1, R27.1, R33.1
- net Filtered_VI: now also U4.16 (PC1), U6.8; no longer C12.2
- net Filtered_VV: now also U4.15 (PC0), U6.14
- net GND: now also C12.2, C21.2, C8.2, C10.2, C13.2, C15.2, C16.2, C17.2, C23.2, C24.2, C26.2, C29.2, C32.2, J1.5 (GND), J1.6 (Shield), J4.13 (Pin_13), J7.3 (Pin_3), R18.2, R8.2, R9.2, SW2.2, U4.10 (VSS), U4.20 (VSSA), U4.27 (VSS), U4.74 (VSS), U4.99 (VSS), U5.4 (V-), U5.5 (+), U6.11 (V-); no longer C21.1, C8.1, R3.2
- net MISO: now also J4.2 (Pin_2), J4.6 (Pin_6), U4.31 (PA6)
- net MOSI: now also J4.3 (Pin_3), J4.9 (Pin_9), U4.32 (PA7)
- net RX: now also J7.2 (Pin_2), R18.1, U4.87 (PD6)
- net SCK: now also J4.5 (Pin_5), J4.8 (Pin_8), U4.30 (PA5)
- net SCL: now also U4.92 (PB6)
- net SDA: now also U4.93 (PB7)
- net SD_CS: now also U4.4 (PE5)
- net STATUS_1: now also U4.81 (PD0)
- net STATUS_2: now also U4.82 (PD1)
- net STATUS_3: now also U4.83 (PD2)
- net TFT_CS: now also J4.12 (Pin_12), U4.1 (PE2)
- net TFT_DC: now also J4.10 (Pin_10), U4.97 (PE0)
- net TFT_RESET: now also J4.11 (Pin_11), U4.98 (PE1)
- net TOUCH_CS: now also J4.4 (Pin_4), U4.3 (PE4)
- net TOUCH_IRQ: now also J4.1 (Pin_1), U4.2 (PE3)
- net TX: now also J7.1 (Pin_1), U4.86 (PD5)
- net at C34.1, R24.1: now also U6.3 (+)
- net at C27.1, R25.2, R28.1: now also U6.1
- net at R28.2, R31.1: now also U6.2 (-)
- net at C35.1, R26.1: now also U6.12 (+)
- net at R29.2, R32.1: now also U6.13 (-)
- net at C51.1, R36.1: now also U6.5 (+)
- net at C39.1, R37.2, R41.1: now also U6.7
- net at R41.2, R43.1: now also U6.6 (-)
- net at C52.1, R38.1: now also U6.10 (+)
- net at R42.2, R44.1: now also U6.9 (-)
- net USB_ID: now reaches R3.1
- net USB_ID: now also U4.69 (PA10); no longer C9.1
- net OSC1: now reaches C31.1
- net OSC1: now also Y2.1, U4.12 (PH0)
- net OSC2: now reaches Y2.2
- net OSC2: now also C32.1, U4.13 (PH1)
- net at R27.2, R30.1: now also U5.3 (+)
- net 2.5V renamed 1.65V
- net 1.65V: now also U5.1, U5.2 (-)
- net RESET: no longer names the net of SW1.1
- net RESET: now also R17.2, R19.1
- new net: U5.6 (-), U5.7
- new net: R8.1, U4.37 (PB2)
- new net: R9.1, U4.91 (PB5)
- new net: J1.4 (ID), R3.2
- new net: J4.7 (Pin_7), R21.1
- new net BOOT0: R19.2, U4.94 (BOOT0)
- new net NRST: C29.1, SW2.1, U4.14 (NRST)
- new net PE10: J3.4 (Pin_4), U4.41 (PE10)
- new net PE11: J3.3 (Pin_3), U4.42 (PE11)
- new net PE12: J3.2 (Pin_2), U4.43 (PE12)
- new net PE13: J3.1 (Pin_1), U4.44 (PE13)
- new net PE6: J3.8 (Pin_8), U4.5 (PE6)
- new net PE7: J3.7 (Pin_7), U4.38 (PE7)
- new net PE8: J3.6 (Pin_6), U4.39 (PE8)
- new net PE9: J3.5 (Pin_5), U4.40 (PE9)
- new net USB_DM: J1.2 (D-), U4.70 (PA11)
- new net USB_DP: J1.3 (D+), U4.71 (PA12)
- new net VBUS: C8.1, J1.1 (VBUS), U4.68 (PA9)
- new net VCAP_1: C9.1, U4.49 (VCAP_1)
- new net VCAP_2: C10.1, U4.73 (VCAP_2)
- no-connect marks 10 -> 5
Other:
- note removed: "Connections"
- note removed: "MCU"
- note removed: "Peak Detectors"
- note removed: "Phase Detector"
- moved on the sheet: D1, D2, D3, J5, R12, R13, R14, TP1, TP2
